File: Kicad/project/SommerESP.kicad_pcb (KiCad board)
At the start: 2 copper layers, 50.7 x 48.6 mm, 43 parts, among them J1 Serial programmer, J2 BRIDGE CONEX, J3 SOMMER CONEX BOARD, J4 SOMMER CONEX KEYPAD, J5 BRIDGE POWER, J6 SOMMER OUTPUT OC, Q1 STN3NF06, U2 G3VM-61D1, U3 G3VM-61D1, U4 LM2596SX-3.3/NOPB, U5 ESP32-C3-WROOM-02

Commit message: Added instructions
Other:
- board text added: "SommerESP v1 Control board"
- board text added: "SommerESP v1 Power board"
- board text removed: "SommerESP v0.1 PSU board"
- board text removed: "SommerESP v0.3 Control board"
Changed lines of the file:
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@@
     (fp_line (start 7.45 3.4) (end 7.45 -2.35)
       (stroke (width 0.1) (type solid)) (layer "F.Fab"))
-    (pad "1" thru_hole roundrect (at 0 0 270) (size 1.7 1.95) (drill 0.95) (layers "*.Cu" "*.Mask") (roundrect_rratio 0.147059)
+    (pad "1" thru_hole roundrect (at 0 0 270) (size 1.7 1.95) (drill 0.95) (layers "*.Cu" "*.Mask") (roundrect_rratio 0.1470588235)
       (net 6 "GND2") (pinfunction "Pin_1") (pintype "passive"))
     (pad "2" thru_hole oval (at 2.5 0 270) (size 1.7 1.95) (drill 0.95) (layers "*.Cu" "*.Mask")
@@
     (fp_line (start 1.6 0.8) (end -1.6 0.8)
       (stroke (width 0.1) (type solid)) (layer "F.Fab"))
-    (pad "1" smd roundrect (at -1.5625 0 180) (size 1.325 1.8) (layers "F.Cu" "F.Paste" "F.Mask") (roundrect_rratio 0.188679)
+    (pad "1" smd roundrect (at -1.5625 0 180) (size 1.325 1.8) (layers "F.Cu" "F.Paste" "F.Mask") (roundrect_rratio 0.1886792453)
       (net 15 "+3.3VA") (pintype "passive"))
-    (pad "2" smd roundrect (at 1.5625 0 180) (size 1.325 1.8) (layers "F.Cu" "F.Paste" "F.Mask") (roundrect_rratio 0.188679)
+    (pad "2" smd roundrect (at 1.5625 0 180) (size 1.325 1.8) (layers "F.Cu" "F.Paste" "F.Mask") (roundrect_rratio 0.1886792453)
       (net 6 "GND2") (pintype "passive"))
     (model "${KICAD6_3DMODEL_DIR}/Capacitor_SMD.3dshapes/C_1206_3216Metric.wrl"
@@
     (fp_line (start 7.45 3.4) (end 7.45 -2.35)
       (stroke (width 0.1) (type solid)) (layer "F.Fab"))
-    (pad "1" thru_hole roundrect (at 0 0 270) (size 1.7 1.95) (drill 0.95) (layers "*.Cu" "*.Mask") (roundrect_rratio 0.147059)
+    (pad "1" thru_hole roundrect (at 0 0 270) (size 1.7 1.95) (drill 0.95) (layers "*.Cu" "*.Mask") (roundrect_rratio 0.1470588235)
       (net 4 "+3.3V") (pinfunction "Pin_1") (pintype "passive"))
     (pad "2" thru_hole oval (at 2.5 0 270) (size 1.7 1.95) (drill 0.95) (layers "*.Cu" "*.Mask")
@@
   (gr_line (start 107.2 90.2) (end 118.9 90.2)
     (stroke (width 0.1) (type default)) (layer "Edge.Cuts"))
-  (gr_text "SommerESP v0.3\nControl board" (at 126.975 72.525 90) (layer "B.SilkS")
+  (gr_text "SommerESP v1\nControl board" (at 126.975 72.525 90) (layer "B.SilkS")
     (effects (font (size 1.5 1.5) (thickness 0.3) bold) (justify bottom mirror))
   )
@@
     (effects (font (size 1 1) (thickness 0.15)) (justify left bottom mirror))
   )
-  (gr_text "SommerESP v0.1\nPSU board" (at 92.575 63.725 270) (layer "B.SilkS")
+  (gr_text "SommerESP v1\nPower board" (at 92.575 63.725 270) (layer "B.SilkS")
     (effects (font (size 1.5 1.5) (thickness 0.3) bold) (justify bottom mirror))
   )
