File: Kicad/SommerESP/SommerESP.kicad_sch (KiCad schematic)
At the start: 29 parts, among them J1 Serial programmer, J3 SOMMER CONEX BOARD, J4 SOMMER CONEX KEYPAD, J6 SOMMER OUTPUT OC, Q1 STN3NF06, Q2 2N7002DW, U4 LM2596SX-3.3/NOPB, U5 ESP32-C3-WROOM-02

Commit message: Fixed wrong LCSC number on the BOM
Parts:
- C1: LCSC C412252 -> C307525
- C2: LCSC C412252 -> C5137467
- C4: LCSC C412252 -> C5674

Commit message: Added 7.5mm position for J7 for more compatibility and updated the readme
Parts:
- added J7: SOMMER OUTPUT OC 7.5mm, Connector_PinSocket_2.54mm:PinSocket_1x04_P2.54mm_Vertical, symbol Connector:Conn_01x04_Female
- C1: LCSC C307525 -> (none); LCSC PN (none) -> C307525
- C2: LCSC C5137467 -> (none); LCSC PN (none) -> C5137467
- C3: LCSC C412252 -> (none); LCSC PN (none) -> C412252
- C4: LCSC C5674 -> (none); LCSC PN (none) -> C5674
- D1: LCSC C397047 -> (none); LCSC PN (none) -> C397047
- D2: LCSC C497961 -> (none); LCSC PN (none) -> C497961
- D3: LCSC C5449114 -> (none); LCSC PN (none) -> C5449114
- D4: LCSC C402212 -> (none); LCSC PN (none) -> C917030
- D5: LCSC C2902914 -> (none); LCSC PN (none) -> C2902914
- J1: LCSC PN (none) -> C6332201
- J3: LCSC C146243 -> (none); LCSC PN (none) -> C146243
- J4: LCSC C49257 -> (none); LCSC PN (none) -> C49257
- J6: LCSC C2718488 -> (none); LCSC PN (none) -> C2718488
- L1: LCSC C7461364 -> (none); LCSC PN (none) -> C7461364
- Q1: LCSC C222218 -> (none); LCSC PN (none) -> C222218
- Q2: LCSC PN (none) -> C5190214
- R1, R2: LCSC C3017758 -> (none); LCSC PN (none) -> C3017758
- R11, R7, R8: LCSC C116692 -> (none); LCSC PN (none) -> C116692
- R12, R13, R3, R4: LCSC C2930027 -> (none); LCSC PN (none) -> C2930027
- S1, S2: LCSC C2905192 -> (none); LCSC PN (none) -> C2905192
- U4: LCSC C5186052 -> (none); LCSC PN (none) -> C5186052
- U5: LCSC C2934560 -> (none); LCSC PN (none) -> C2934560
Connections:
- net +24V: now also J7.1 (Pin_1)
- net GND: now also J7.4 (Pin_4)
- net SommerSIG: now also J7.3 (Pin_3)
- no-connect marks 1 -> 2

Commit message: Added fabrication holes on the PCB and setup up for production.
Parts:
- added H1, H2, H3: MountingHole, MountingHole:ToolingHole_1.152mm, symbol Mechanical:MountingHole
- added J8: SOMMER OUTPUT OC 8.5mm, SommerCustom:PinSocket_1x04_P2.54mm_Vertical_SLIT, symbol Connector:Conn_01x04_Female
- added TP1: TestPoint, TestPoint:TestPoint_Pad_2.0x2.0mm, symbol Connector:TestPoint
- J6: value SOMMER OUTPUT OC -> SOMMER OUTPUT OC 9.5; footprint Connector_PinSocket_2.54mm:PinSocket_1x04_P2.54mm_Vertical -> SommerCustom:PinSocket_1x04_P2.54mm_Vertical_SLIT
- J7: footprint Connector_PinSocket_2.54mm:PinSocket_1x04_P2.54mm_Vertical -> SommerCustom:PinSocket_1x04_P2.54mm_Vertical_SLIT
Connections:
- net +24V: now also J8.1 (Pin_1)
- net GND: now also J8.4 (Pin_4)
- net SommerSIG: now also J8.3 (Pin_3)
- net at R1.1, S1.1: now also TP1.1
- no-connect marks 2 -> 3
Other:
- title: (none) -> SommerESP
- moved on the sheet: J6, J7

Commit message: Added RST pad
Parts:
- added TP2: RST, TestPoint:TestPoint_Pad_2.0x2.0mm, symbol Connector:TestPoint
- TP1: value TestPoint -> BOOT
Connections:
- net at R2.1, S2.1: now also TP2.1
Changed lines of the file:
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@@
 		(color 0 0 0 0)
 	)
+	(junction
+		(at 38.1 104.14)
+		(diameter 0)
+		(color 0 0 0 0)
+	)
 	(no_connect
 		(at 189.23 68.58)
@@
 	(wire
 		(pts
+			(xy 38.1 97.79) (xy 38.1 104.14)
+		)
+		(stroke
+			(width 0)
+			(type default)
+		)
+	)
+	(wire
+		(pts
 			(xy 102.87 101.6) (xy 109.22 101.6)
 		)
@@
 	)
 	(symbol
+		(lib_id "Connector:TestPoint")
+		(at 38.1 97.79 0)
+		(unit 1)
+		(body_style 1)
+		(exclude_from_sim no)
+		(in_bom yes)
+		(on_board yes)
+		(in_pos_files yes)
+		(dnp no)
+		(fields_autoplaced yes)
+		(property "Reference" "TP2"
+			(at 40.64 93.2179 0)
+			(show_name no)
+			(do_not_autoplace no)
+			(effects
+				(font
+					(size 1.27 1.27)
+				)
+				(justify left)
+			)
+		)
+		(property "Value" "RST"
+			(at 40.64 95.7579 0)
+			(show_name no)
+			(do_not_autoplace no)
+			(effects
+				(font
+					(size 1.27 1.27)
+				)
+				(justify left)
+			)
+		)
+		(property "Footprint" "TestPoint:TestPoint_Pad_2.0x2.0mm"
+			(at 43.18 97.79 0)
+			(hide yes)
+			(show_name no)
+			(do_not_autoplace no)
+			(effects
+				(font
+					(size 1.27 1.27)
+				)
+			)
+		)
+		(property "Datasheet" ""
+			(at 43.18 97.79 0)
+			(hide yes)
+			(show_name no)
+			(do_not_autoplace no)
+			(effects
+				(font
+					(size 1.27 1.27)
+				)
+			)
+		)
+		(property "Description" "test point"
+			(at 38.1 97.79 0)
+			(hide yes)
+			(show_name no)
+			(do_not_autoplace no)
+			(effects
+				(font
+					(size 1.27 1.27)
+				)
+			)
+		)
+		(pin "1"
+		)
+		(instances
+			(project "SommerESP"
+				(path "/fdfaab82-b631-42c7-9b66-01e568778cad"
+					(reference "TP2")
+					(unit 1)
+				)
+			)
+		)
+	)
+	(symbol
 		(lib_id "Connector:Conn_01x04_Female")
 		(at 184.15 48.26 180)
@@
 			)
 		)
-		(property "Value" "TestPoint"
+		(property "Value" "BOOT"
 			(at 40.64 74.1679 0)
 			(show_name no)
